Commit message: delete body

File: envs/GankenKun_pybullet/URDF/gankenkun.urdf (robot description, URDF)
Before this commit: robot gankenkun, 35 links, 34 joints
Links:
- link body_link: geometry 
- link head_yaw_link: geometry 
- link left_lower_arm_link: geometry 
- link left_shin_pitch_link: geometry 
- link left_shin_pitch_mimic_link: geometry 
- link left_shoulder_link: geometry 
- link left_slider_crank_link: geometry 
- link left_upper_arm_link: geometry 
- link left_waist_pitch_link: geometry 
- link left_waist_pitch_mimic_link: geometry 
- link left_waist_roll_link: geometry 
- link left_waist_yaw_link: geometry 
- link right_lower_arm_link: geometry 
- link right_shin_pitch_link: geometry 
- link right_shin_pitch_mimic_link: geometry 
- link right_shoulder_link: geometry 
- link right_slider_crank_link: geometry 
- link right_upper_arm_link: geometry 
- link right_waist_pitch_link: geometry 
- link right_waist_pitch_mimic_link: geometry 
- link right_waist_roll_link: geometry 
- link right_waist_yaw_link: geometry 
